File: hardware/kicad/changer cable breakout/changer cable breakout.kicad_sch (KiCad schematic)
At the start: 0 parts

Commit message: make schematic and start layout
Parts:
- added J1, J2: SDD-130J, Library:CUI_SDD-130J, symbol kenwood_changer_emulator:SDD-130J
- added J3: Test Points, Connector_PinSocket_2.54mm:PinSocket_2x07_P2.54mm_Vertical, symbol Connector_Generic:Conn_02x07_Counter_Clockwise
Connections:
- new net B.U.: J1.3, J2.3, J3.3 (Pin_3)
- new net D. GND: J1.6, J2.6, J3.6 (Pin_6)
- new net DATA C: J1.10, J2.10, J3.10 (Pin_10)
- new net DATA H: J1.11, J2.11, J3.11 (Pin_11)
- new net GND: J1.2, J2.2, J3.2 (Pin_2)
- new net GND1: J1.E1 (GND), J1.E2 (GND__1), J2.E1 (GND), J2.E2 (GND__1)
- new net L CH: J1.12, J2.12, J3.12 (Pin_12)
- new net MUTE: J1.5, J2.5, J3.5 (Pin_5)
- new net ON: J1.4, J2.4, J3.4 (Pin_4)
- new net RESET: J1.7, J2.7, J3.7 (Pin_7)
- new net R_CH: J1.8, J2.8, J3.8 (Pin_8)
- new net ~{CLK}: J1.13, J2.13, J3.13 (Pin_13)
- new net ~{REQ_C}: J1.9, J2.9, J3.9 (Pin_9)
- new net ~{REQ_H}: J1.1, J2.1, J3.1 (Pin_1)
- no-connect marks 0 -> 1
Other:
- title: (none) -> 13 PIN MINI DIN BREAKOUT PASSTHROUGH

Commit message: finish breakout design
Parts:
- removed J3: Test Points, Connector_PinSocket_2.54mm:PinSocket_2x07_P2.54mm_Vertical, symbol Connector_Generic:Conn_02x07_Counter_Clockwise
- added J3: Test Points, Library:PinSocket_1x11_P2.54mm_Vertical, symbol Connector:Conn_01x11_Socket
- added J4, J5: AudioJack3, Library:Jack_3.5mm_CUI_SJ1-3523N_Horizontal, symbol Connector_Audio:AudioJack3
Connections:
- net B.U.: now also J3.3 (Pin_3)
- net D. GND: now also J3.5 (Pin_5)
- net DATA C: now also J3.9 (Pin_9)
- net DATA H: now also J3.10 (Pin_10)
- net GND: now also J3.1 (Pin_1), J4.S, J5.S
- net MUTE: now also J3.8 (Pin_8)
- net ON: now also J3.2 (Pin_2)
- net RESET: now also J3.4 (Pin_4)
- net ~{CLK}: now also J3.11 (Pin_11)
- net ~{REQ_C}: now also J3.7 (Pin_7)
- net ~{REQ_H}: now also J3.6 (Pin_6)
- net L CH renamed L_ch_C
- net L_ch_C: now also J5.R; no longer J1.12
- net R_CH renamed R_ch_C
- net R_ch_C: now also J5.T; no longer J1.8
- new net L_ch_H: J1.12, J4.R
- new net R_ch_H: J1.8, J4.T
- no-connect marks 1 -> 0
Other:
- note added: "Changer Side"
- note added: "Head Unit Side"
