File: hardware/kicad/emulator hat/emulator hat.kicad_sch (KiCad schematic)
At the start: 0 parts

Commit message: begin hat design
Parts:
- added C1, C10, C3, C5: 10uF, symbol Device:C_Polarized_Small
- added C11, C12: 2.2nF, Capacitor_SMD:C_0603_1608Metric_Pad1.08x0.95mm_HandSolder, symbol Device:C_Small
- added C2, C4, C6, C9: .1uF, Capacitor_SMD:C_0603_1608Metric_Pad1.08x0.95mm_HandSolder, symbol Device:C_Small
- added C7, C8: 2.2uF, Capacitor_SMD:C_0603_1608Metric_Pad1.08x0.95mm_HandSolder, symbol Device:C_Small
- added D1: D_Schottky, Diode_SMD:D_0603_1608Metric_Pad1.05x0.95mm_HandSolder, symbol Device:D_Schottky
- added J1: SDD-130J, Library:CUI_SDD-130J, symbol kenwood_changer_emulator:SDD-130J_CHANGER_PORT
- added J3: Raspberry_Pi_4, Connector_PinSocket_2.54mm:PinSocket_2x20_P2.54mm_Vertical, symbol Connector:Raspberry_Pi_4
- added R1: 47K, Resistor_SMD:R_0603_1608Metric_Pad0.98x0.95mm_HandSolder, symbol Device:R_Small
- added R2, R3, R4: 470, Resistor_SMD:R_0603_1608Metric_Pad0.98x0.95mm_HandSolder, symbol Device:R_Small
- added U1: ATtiny1616-M, Package_DFN_QFN:VQFN-20-1EP_3x3mm_P0.4mm_EP1.7x1.7mm_ThermalVias, symbol MCU_Microchip_ATtiny:ATtiny1616-M
- added U2: PCM5102A, Package_SO:TSSOP-20_4.4x6.5mm_P0.65mm, symbol Audio:PCM5102A
- added U3, U4: SN74LVC8T245, Package_SO:SSOP-24_5.3x8.2mm_P0.65mm, symbol kenwood_changer_emulator:SN74LVC8T245_MOD
Connections:
- new net: C7.1, U2.2 (CAPP)
- new net: C7.2, U2.4 (CAPM)
- new net: C8.1, U2.5 (VNEG)
- new net: R3.1, U2.7 (OUTR)
- new net: C10.1, C9.1, U2.18 (LDOO)
- new net: R2.1, U2.6 (OUTL)
- new net: R1.2, U2.17 (XSMT)
- new net +3.3V: C3.1, C4.1, J3.1 (3V3), J3.17 (3V3), R1.1, U1.4 (VCC), U2.20 (DVDD)
- new net +3.3VA: C1.1, C2.1, C5.1, C6.1, U2.1 (CPVDD), U2.8 (AVDD)
- new net +5V: J3.2 (5V), J3.4 (5V)
- new net BCK: J3.12 (GPIO18/SPI1_~{CE0}/PCM_CLK/PWM0), U2.13 (BCK)
- new net BUS_DATA_C: J1.10 (DATA_C), U4.3 (A1)
- new net BUS_DATA_H: J1.11 (DATA_H), U3.4 (A2)
- new net BUS_MUTE: J1.5 (MUTE), U4.5 (A3)
- new net BUS_ON: J1.4 (ON), U3.6 (A4)
- new net BUS_RESET: J1.7 (RESET), U3.7 (A5)
- new net BUS_~{CLK}: J1.13 (~{CLK}), U3.3 (A1)
- new net BUS_~{REQ_C}: J1.9 (~{REQ_C}), U4.4 (A2)
- new net BUS_~{REQ_H}: J1.1 (~{REQ_H}), U3.5 (A3)
- new net DATA C: U1.6 (PA5), U4.21 (B1)
- new net DATA H: U1.5 (PA4), U3.20 (B2)
- new net DIN: J3.40 (GPIO21/SPI1_SCLK/PCM_DOUT), U2.14 (DIN)
- new net GND: C10.2, C3.2, C4.2, C9.2, J1.2 (GND), J1.S (SHIELD), J3.14 (GND), J3.20 (GND), J3.25 (GND), J3.30 (GND), J3.34 (GND), J3.39 (GND), J3.6 (GND), J3.9 (GND), U1.21 (GND), U1.3 (GND), U2.10 (DEMP), U2.11 (FLT), U2.12 (SCK), U2.16 (FMT), U2.19 (DGND), U3.10 (A8), U3.11 (GND), U3.12 (GND), U3.13 (GND), U3.8 (A6), U3.9 (A7), U4.10 (A8), U4.11 (GND), U4.12 (GND), U4.13 (GND), U4.6 (A4), U4.7 (A5), U4.8 (A6), U4.9 (A7)
- new net GNDA: C1.2, C11.2, C12.2, C2.2, C5.2, C6.2, C8.2, J1.6 (AGND), U2.3 (CPGND), U2.9 (AGND)
- new net LRCK: J3.35 (GPIO19/SPI1_MISO/PCM_FS), U2.15 (LRCK)
- new net L_ch: C11.1, J1.12 (L_ch), R2.2
- new net MUTE: U1.13 (PB1), U4.19 (B3)
- new net ON: U1.14 (PB0), U3.18 (B4)
- new net RESET: U1.12 (PB2), U3.17 (B5)
- new net RX3: D1.1 (K), J3.29 (GPCLK1/GPIO05)
- new net R_ch: C12.1, J1.8 (R_ch), R3.2
- new net TX3: J3.7 (GPCLK0/GPIO04), R4.2
- new net UART_RX: J3.8 (GPIO14/UART_TXD), U1.1 (PA2)
- new net UART_TX: J3.10 (GPIO15/UART_RXD), U1.20 (PA1)
- new net UPDI: D1.2 (A), R4.1, U1.19 (~{RESET}/PA0)
- new net VBUS: J1.3 (BU+14V)
- new net ~{CLK}: U1.2 (PA3), U3.21 (B1)
- new net ~{REQ_C}: U1.8 (PA7), U4.20 (B2)
- new net ~{REQ_H}: U1.7 (PA6), U3.19 (B3)
- no-connect marks 0 -> 8
Other:
- note added: "13 Pin Mini-DIN Connector"
- note added: "ATtiny1616"
- note added: "Level Shifting"
- note added: "PCM5102A I2S DAC"
